Commit message: add mecanum description and gazebo in empty world

File: mecanum_description/urdf/mecanum_properties.urdf.xacro (robot description, xacro)
@@ -13,5 +13,5 @@
   <xacro:property name="wheel_torque" value="20" />
   <xacro:property name="laser_pose">
-    <origin xyz="-0.0475 0 0.125" rpy="0 0 0"/>
+    <origin xyz="0.0475 0 0.125" rpy="0 0 0"/>
   </xacro:property>
 </robot>

File: mecanum_description/urdf/mecanum_robot.urdf.xacro (robot description, xacro)
@@ -50,5 +50,5 @@
     mass="${wheel_mass}"
   />
-  <xacro:imu/>
+  <!-- <xacro:imu/> -->
   <xacro:generic_laser>
     <xacro:insert_block name="laser_pose" />
