Commit message: update for Course SLAM

File: mecanum_description/urdf/basic_mobile_robot.urdf.xacro (robot description, xacro)
@@ -66,7 +66,4 @@
     <xacro:box_inertia m="40.0" w="${base_width}" d="${base_length}" h="${base_height}"/>
   </link>
-  <gazebo reference="base_link">
-    <material>Gazebo/Red</material>
-  </gazebo>
   <!-- *********************** DRIVE WHEELS ******************************  -->
   <xacro:macro name="wheel" params="prefix x_reflect y_reflect">
@@ -126,4 +123,48 @@
     <xacro:sphere_inertia m="10.05" r="${(wheel_radius+wheel_zoff-(base_height/2))}"/>
   </link>
+  <joint name="caster_joint" type="fixed">
+    <parent link="base_link"/>
+    <child link="front_caster"/>
+    <origin xyz="${caster_xoff} 0.0 ${-(base_height/2)}" rpy="0 0 0"/>
+  </joint>
+        <joint name="laser_joint" type="fixed">
+        <parent link="base_link"/>
+        <child link="laser_frame"/>
+        <origin xyz="0.1 0 0.175" rpy="0 0 0"/>
+    </joint>
+    <link name="base_scan">
+        <visual>
+            <geometry>
+                <cylinder radius="0.05" length="0.04"/>
+            </geometry>
+            <material name="red"/>
+        </visual>
+        <collision>
+            <geometry>
+                <cylinder radius="0.05" length="0.04"/>
+            </geometry>
+        </collision>
+        <xacro:cylinder_inertia m="0.1" r="0.05" h="0.04" >
+            <origin xyz="0 0 0" rpy="0 0 0"/>
+        </xacro:cylinder_inertia>
+    </link>
+  <!-- *********************** IMU SETUP *********************************  -->
+  <!-- Each sensor must be attached to a link.                              -->
+  <!-- <joint name="imu_joint" type="fixed">
+    <parent link="base_link"/>
+    <child link="imu_link"/>
+    <origin xyz="-0.10 0 0.05" rpy="0 0 0"/>
+  </joint>
+  <link name="imu_link"/> -->
+  <!-- *********************** GPS SETUP **********************************  -->
+  <!-- <joint name="gps_joint" type="fixed">
+    <parent link="base_link"/>
+    <child link="gps_link"/>
+    <origin xyz="0.10 0 0.05" rpy="0 0 0"/>
+  </joint>
+  <link name="gps_link"/> -->
+  <gazebo reference="base_link">
+    <material>Gazebo/Red</material>
+  </gazebo>
   <gazebo reference="front_caster">
     <mu1>0.01</mu1>
@@ -131,23 +172,49 @@
     <material>Gazebo/White</material>
   </gazebo>
-  <joint name="caster_joint" type="fixed">
-    <parent link="base_link"/>
-    <child link="front_caster"/>
-    <origin xyz="${caster_xoff} 0.0 ${-(base_height/2)}" rpy="0 0 0"/>
-  </joint>
-  <!-- *********************** IMU SETUP *********************************  -->
-  <!-- Each sensor must be attached to a link.                              -->
-  <joint name="imu_joint" type="fixed">
-    <parent link="base_link"/>
-    <child link="imu_link"/>
-    <origin xyz="-0.10 0 0.05" rpy="0 0 0"/>
-  </joint>
-  <link name="imu_link"/>
-  <!-- *********************** GPS SETUP **********************************  -->
-  <joint name="gps_joint" type="fixed">
-    <parent link="base_link"/>
-    <child link="gps_link"/>
-    <origin xyz="0.10 0 0.05" rpy="0 0 0"/>
-  </joint>
-  <link name="gps_link"/>
+  <gazebo>
+    <plugin name="diff_drive" filename="libgazebo_ros_diff_drive.so">
+        <!-- Wheel Information -->
+        <left_joint>left_wheel_joint</left_joint>
+        <right_joint>right_wheel_joint</right_joint>
+        <wheel_separation>0.35</wheel_separation>
+        <wheel_diameter>0.1</wheel_diameter>
+        <!-- Limits -->
+        <max_wheel_torque>200</max_wheel_torque>
+        <max_wheel_acceleration>10.0</max_wheel_acceleration>
+        <!-- Output -->
+        <odometry_frame>odom</odometry_frame>
+        <robot_base_frame>base_link</robot_base_frame>
+        <publish_odom>true</publish_odom>
+        <publish_odom_tf>true</publish_odom_tf>
+        <publish_wheel_tf>true</publish_wheel_tf>
+    </plugin>
+  </gazebo>
+    <gazebo reference="base_scan">
+        <material>Gazebo/Red</material>
+        <sensor name="laser" type="ray">
+            <pose> 0 0 0 0 0 0 </pose>
+            <visualize>true</visualize>
+            <update_rate>10</update_rate>
+            <ray>
+                <scan>
+                    <horizontal>
+                        <samples>360</samples>
+                        <min_angle>-3.14</min_angle>
+                        <max_angle>3.14</max_angle>
+                    </horizontal>
+                </scan>
+                <range>
+                    <min>0.3</min>
+                    <max>12</max>
+                </range>
+            </ray>
+            <plugin name="laser_controller" filename="libgazebo_ros_ray_sensor.so">
+                <ros>
+                    <argument>~/out:=scan</argument>
+                </ros>
+                <output_type>sensor_msgs/LaserScan</output_type>
+                <frame_name>laser_frame</frame_name>
+            </plugin>
+        </sensor>
+    </gazebo>
 </robot>

File: mecanum_description/urdf/generic_laser.urdf.xacro (robot description, xacro)
@@ -10,5 +10,5 @@
       min_range="0.08"
       max_range="12.0"
-      frame_id="laser"
+      frame_id="base_scan"
       topic_name="scan"
     >

File: mecanum_description/urdf/mecanum_drive.urdf.xacro (robot description, xacro)
@@ -9,8 +9,9 @@
       <odometry_topic>odom</odometry_topic>
       <odometry_frame>odom</odometry_frame>
-      <odometry_rate>20.0</odometry_rate>
+      <odometry_rate>50.0</odometry_rate>
       <robot_base_frame>base_footprint</robot_base_frame>
       <publish_odom>true</publish_odom>
       <publish_odom_tf>true</publish_odom_tf>
+      <publish_wheel_tf>true</publish_wheel_tf>
     </plugin>
   </gazebo>

File: mecanum_description/urdf/mecanum_wheel.urdf.xacro (robot description, xacro)
@@ -40,5 +40,5 @@
       </visual>
     </gazebo>
-    <joint name="${side}_wheel_joint" type="continuous">
+    <joint name="${side}_wheel_joint" type="fixed">
       <axis xyz="0 1 0" />
       <parent link="base_link"/>
